File: mainboard/mainboard.kicad_pcb (KiCad board)
At the start: 2 copper layers, 0 parts

Commit message: edge cuts work
Other:
- board outline added: 260 x 146 mm
Changed lines of the file:
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@@
 		(stroke
 			(width 0.1)
-			(type default)
-		)
-		(layer "F.Fab")
+			(type solid)
+		)
+		(layer "Edge.Cuts")
 	)
 	(gr_line
@@
 		(stroke
 			(width 0.1)
-			(type default)
-		)
-		(layer "F.Fab")
+			(type solid)
+		)
+		(layer "Edge.Cuts")
 	)
 	(gr_line
@@
 		(stroke
 			(width 0.1)
-			(type default)
-		)
-		(layer "F.Fab")
+			(type solid)
+		)
+		(layer "Edge.Cuts")
 	)
 	(gr_line
@@
 		(stroke
 			(width 0.1)
-			(type default)
-		)
-		(layer "F.Fab")
+			(type solid)
+		)
+		(layer "Edge.Cuts")
 	)
 	(gr_line
@@
 		(stroke
 			(width 0.1)
-			(type default)
-		)
-		(layer "F.Fab")
+			(type solid)
+		)
+		(layer "Edge.Cuts")
 	)
 	(gr_line
@@
 		(stroke
 			(width 0.1)
-			(type default)
-		)
-		(layer "F.Fab")
+			(type solid)
+		)
+		(layer "Edge.Cuts")
 	)
 	(gr_line
@@
 		(stroke
 			(width 0.1)
-			(type default)
-		)
-		(layer "F.Fab")
+			(type solid)
+		)
+		(layer "Edge.Cuts")
 	)
 	(gr_line
@@
 		(stroke
 			(width 0.1)
-			(type default)
-		)
-		(layer "F.Fab")
+			(type solid)
+		)
+		(layer "Edge.Cuts")
 	)
 	(gr_line
@@
 		(stroke
 			(width 0.1)
-			(type default)
-		)
-		(layer "F.Fab")
+			(type solid)
+		)
+		(layer "Edge.Cuts")
 	)
 	(gr_line
@@
 		(stroke
 			(width 0.1)
-			(type default)
-		)
-		(layer "F.Fab")
+			(type solid)
+		)
+		(layer "Edge.Cuts")
 	)
 	(gr_line
@@
 		(stroke
 			(width 0.1)
-			(type default)
-		)
-		(layer "F.Fab")
+			(type solid)
+		)
+		(layer "Edge.Cuts")
 	)
 	(gr_line
@@
 		(stroke
 			(width 0.1)
-			(type default)
-		)
-		(layer "F.Fab")
+			(type solid)
+		)
+		(layer "Edge.Cuts")
 	)
 	(gr_line
@@
 		(stroke
 			(width 0.1)
-			(type default)
-		)
-		(layer "F.Fab")
+			(type solid)
+		)
+		(layer "Edge.Cuts")
 	)
 	(gr_line
@@
 		(stroke
 			(width 0.1)
-			(type default)
-		)
-		(layer "F.Fab")
+			(type solid)
+		)
+		(layer "Edge.Cuts")
 	)
 	(gr_line
@@
 		(stroke
 			(width 0.1)
-			(type default)
-		)
-		(layer "F.Fab")
+			(type solid)
+		)
+		(layer "Edge.Cuts")
 	)
 	(gr_line
@@
 		(stroke
 			(width 0.1)
-			(type default)
-		)
-		(layer "F.Fab")
+			(type solid)
+		)
+		(layer "Edge.Cuts")
 	)
 	(gr_line
@@
 		(stroke
 			(width 0.1)
-			(type default)
-		)
-		(layer "F.Fab")
+			(type solid)
+		)
+		(layer "Edge.Cuts")
 	)
 	(gr_line
@@
 		(stroke
 			(width 0.1)
-			(type default)
-		)
-		(layer "F.Fab")
+			(type solid)
+		)
+		(layer "Edge.Cuts")
 	)
 	(gr_line
@@
 		(stroke
 			(width 0.1)
-			(type default)
-		)
-		(layer "F.Fab")
+			(type solid)
+		)
+		(layer "Edge.Cuts")
 	)
 	(gr_line
@@
 		(stroke
 			(width 0.1)
-			(type default)
-		)
-		(layer "F.Fab")
+			(type solid)
+		)
+		(layer "Edge.Cuts")
 	)
 	(gr_line
@@
 		(stroke
 			(width 0.1)
-			(type default)
-		)
-		(layer "F.Fab")
+			(type solid)
+		)
+		(layer "Edge.Cuts")
 	)
 	(gr_line
@@
 		(stroke
 			(width 0.1)
-			(type default)
-		)
-		(layer "F.Fab")
+			(type solid)
+		)
+		(layer "Edge.Cuts")
 	)
 	(gr_line
@@
 		(stroke
 			(width 0.1)
-			(type default)
-		)
-		(layer "F.Fab")
+			(type solid)
+		)
+		(layer "Edge.Cuts")
 	)
 	(gr_line
@@
 		(stroke
 			(width 0.1)
-			(type default)
-		)
-		(layer "F.Fab")
+			(type solid)
+		)
+		(layer "Edge.Cuts")
 	)
 	(gr_line
@@
 		(stroke
 			(width 0.1)
-			(type default)
-		)
-		(layer "F.Fab")
+			(type solid)
+		)
+		(layer "Edge.Cuts")
 	)
 	(gr_line
@@
 		(stroke
 			(width 0.1)
-			(type default)
-		)
-		(layer "F.Fab")
+			(type solid)
+		)
+		(layer "Edge.Cuts")
 	)
 	(gr_line
@@
 		(stroke
 			(width 0.1)
-			(type default)
-		)
-		(layer "F.Fab")
+			(type solid)
+		)
+		(layer "Edge.Cuts")
 	)
 	(gr_line
@@
 		(stroke
 			(width 0.1)
-			(type default)
-		)
-		(layer "F.Fab")
+			(type solid)
+		)
+		(layer "Edge.Cuts")
 	)
 	(gr_line
@@
 		(stroke
 			(width 0.1)
-			(type default)
-		)
-		(layer "F.Fab")
+			(type solid)
+		)
+		(layer "Edge.Cuts")
 	)
 	(embedded_fonts no)
